Commit message: Stonefish update

File: sam_description/urdf/sam_auv.urdf.xacro (robot description, xacro)
@@ -1,3 +1,3 @@
-<?xml version="2.0"?>
+<?xml version="1.0"?>
 <robot name="sam" xmlns:xacro="http://www.ros.org/wiki/xacro">
   <!-- Meshes. -->
@@ -6,5 +6,5 @@
   <xacro:property name="front_prop" value="file://$(find sam_description)/mesh/SAM_FRONTPROP.dae"/>
   <xacro:property name="back_prop" value="file://$(find sam_description)/mesh/SAM_BACKPROP.dae"/>
-  <xacro:macro name="sam_auv" params="namespace debug">
+  <!-- <xacro:macro name="sam_auv" params="namespace debug"> -->
   <!-- Links. -->
   <link name="$(arg namespace)/base_link">
@@ -160,4 +160,4 @@
     <limit lower="-1.6" upper="1.6" velocity="0.2" effort="1.0"/>
   </joint>
-  </xacro:macro>
+  <!-- </xacro:macro> -->
 </robot>

Commit message: Fixed the rotation (again)

File: sam_description/urdf/sam_auv.urdf.xacro (robot description, xacro)
@@ -121,5 +121,5 @@
     <parent link="$(arg namespace)/base_link"/>
     <child link="$(arg namespace)/camera_front_link"/>
-    <origin rpy="0.0 1.5707 0.0" xyz="0.647 0.0 0.0"/>
+    <origin rpy="-1.5707 0.0 -1.5707" xyz="0.647 0.0 0.0"/>
   </joint>
   <joint name="$(arg namespace)/camera_down_joint" type="fixed">
@@ -131,11 +131,12 @@
     <parent link="$(arg namespace)/base_link"/>
     <child link="$(arg namespace)/camera_front_left_link"/>
-    <!--origin rpy="1.3 3.1416 2.3416" xyz="0.636 0.050 -0.007"/-->
-    <origin rpy="-0.2217 1.7243 0.6039" xyz="0.636 0.050 -0.007"/>
+    <origin rpy="1.3 3.1416 2.3416" xyz="0.636 0.050 -0.007"/>
+    <!-- <origin rpy="-0.2217 1.7243 0.6039" xyz="0.636 0.050 -0.007"/> -->
   </joint>
   <joint name="$(arg namespace)/camera_front_right_joint" type="fixed">
     <parent link="$(arg namespace)/base_link"/>
     <child link="$(arg namespace)/camera_front_right_link"/>
-    <origin rpy="0.2217 1.7243 -0.6039" xyz="0.636 -0.050 -0.007"/>
+    <!-- <origin rpy="0.2217 1.7243 -0.6039" xyz="0.636 -0.050 -0.007"/> -->
+    <origin rpy="1.3 3.1416 0.8" xyz="0.636 -0.050 -0.007"/>
   </joint>
   <joint name="$(arg namespace)/lcg_joint" type="prismatic">
