Commit message: Some update on the camera position

File: cm_station_description/urdf/cm_station.urdf.xacro (robot description, xacro)
@@ -38,5 +38,5 @@
     <parent link="$(arg namespace)/base_link"/>
     <child link="$(arg namespace)/uw_cam_link"/>
-    <origin rpy="0.0 2.76893 0.0" xyz="0.4 0. 0"/>
+    <origin rpy="0.0 2.76893 0.0" xyz="0.4 -0.5 0"/>
     <!-- <origin rpy="0.0 0.698132 0.0" xyz="0.3 0. 0"/> -->
     <!-- <origin rpy="${-pi/2} 0.0 ${-pi/2}" xyz="0.3 0. 0"/> -->
